File: PCB/PowerSupply.kicad_sch (KiCad schematic)
At the start: 35 parts, among them J1 V+, J10 GND, J2 V-, J23 Conn_01x02, J27 SU5V_E+, J28 SU5V_E-, J29 SU5V_A+, J3 U+, J30 SU5V_A-, J31 LED, J32 TP_GND, J33 TP_3,3V, J34 TP_VBAT, J35 TP_12V, J36 TP_5V, J4 U-, J5 B+, J6 B-, J7 SU12_in, J8 GND, J9 SU12_out, U1 AP2112K-3.3

Commit message: Text geändert
Other:
- note added: "Batterie kommt da"
- note removed: "Batterie kommt da dran"
Changed lines of the file:
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@@
 		)
 	)
-	(text "Batterie kommt da dran\n"
+	(text "Batterie kommt da \n"
 		(exclude_from_sim no)
 		(at 106.172 80.264 0)

Commit message: Änderung der PSU
Parts:
- added J37: Boost Schalter, symbol Connector_Generic:Conn_01x02
- added J38: Batterie, symbol Connector_Generic:Conn_01x02
- J23: value Conn_01x02 -> Digitalschalter
Connections:
- net GND: now also J6.1 (Pin_1), J38.2 (Pin_2)
- net U+: no longer C8.1, J34.1 (Pin_1), J7.1 (Pin_1)
- net Bat+: now reaches J5.1 (Pin_1)
- net Bat+: now also J34.1 (Pin_1), J37.1 (Pin_1), J38.1 (Pin_1)
- new net Boost_In: C8.1, J37.2 (Pin_2), J7.1 (Pin_1)
- no-connect marks 4 -> 2
Other:
- note removed: "Batterie kommt da"

Commit message: Schematic letzte Fehler Behebung
Parts:
- J38: value Batterie -> Digital Schalter
Changed lines of the file:
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@@
 			)
 		)
-		(property "Value" "Batterie"
+		(property "Value" "Digital Schalter"
 			(at 129.54 21.5899 90)
 			(show_name no)

Commit message: Implementation of StepDown und 0Ohm Resistors
Parts:
- added C31: 100nF, symbol Device:C
- added R11, R12: 0, symbol Device:R
- J38: value Digital Schalter -> Battery
Connections:
- net +12V: now also R12.2; no longer C4.1, C5.1, C6.1, L1.2
- net +3.3V: now also R11.2; no longer C7.1, U1.5 (VOUT)
- net GND: now also C31.2
- net U+: no longer C28.1, J27.1 (Pin_1)
- net 12V_RAW: now reaches C2.1, C3.1, J9.1 (Pin_1), L1.1
- net 12V_RAW: now also C28.1, J27.1 (Pin_1), C31.1
- new net: C4.1, C5.1, C6.1, L1.2, R12.1
- new net: C7.1, R11.1, U1.5 (VOUT)
Other:
- moved on the sheet: C28

Commit message: Schematic with footprints. ERC okay
Parts:
- C1, C7: footprint (none) -> Capacitor_SMD:C_0805_2012Metric
- C2, C29: footprint (none) -> Capacitor_THT:CP_Radial_D6.3mm_P2.50mm
- C28, C30, C6: footprint (none) -> Capacitor_SMD:C_1206_3216Metric
- C3, C31, C5: footprint (none) -> Capacitor_SMD:C_0603_1608Metric
- C4, C8: footprint (none) -> Capacitor_THT:CP_Radial_D8.0mm_P3.50mm
- J10, J8, J9: footprint (none) -> Connector_Wire:SolderWire-1sqmm_1x01_D1.4mm_OD2.7mm
- J2, J3, J4, J6: footprint (none) -> Connector_PinHeader_2.00mm:PinHeader_1x01_P2.00mm_Vertical
- J31: footprint (none) -> Connector_PinHeader_2.54mm:PinHeader_1x02_P2.54mm_Vertical
- J37, J38: footprint (none) -> Connector_Wire:SolderWire-1sqmm_1x02_P5.4mm_D1.4mm_OD2.7mm
- J7: footprint Connector_PinHeader_2.00mm:PinHeader_1x01_P2.00mm_Vertical -> Connector_Wire:SolderWire-1sqmm_1x01_D1.4mm_OD2.7mm
- L1: footprint (none) -> Inductor_SMD:L_Bourns_SRR1260
- R10, R11: footprint (none) -> Resistor_SMD:R_0603_1608Metric
- R12: footprint (none) -> Resistor_THT:R_Axial_DIN0207_L6.3mm_D2.5mm_P10.16mm_Horizontal
Changed lines of the file:
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@@
 	)
 	(junction
+		(at 95.25 166.37)
+		(diameter 0)
+		(color 0 0 0 0)
+	)
+	(junction
 		(at 91.44 27.94)
 		(diameter 0)
@@
 	(wire
 		(pts
+			(xy 95.25 166.37) (xy 97.79 166.37)
+		)
+		(stroke
+			(width 0)
+			(type default)
+		)
+	)
+	(wire
+		(pts
 			(xy 50.8 50.8) (xy 50.8 54.61)
 		)
@@
 	(wire
 		(pts
-			(xy 91.44 166.37) (xy 97.79 166.37)
+			(xy 91.44 166.37) (xy 95.25 166.37)
 		)
 		(stroke
@@
 	(wire
 		(pts
+			(xy 95.25 166.37) (xy 95.25 171.45)
+		)
+		(stroke
+			(width 0)
+			(type default)
+		)
+	)
+	(wire
+		(pts
 			(xy 97.79 106.68) (xy 97.79 113.03)
 		)
@@
 			)
 		)
-		(property "Footprint" ""
+		(property "Footprint" "Capacitor_THT:CP_Radial_D8.0mm_P3.50mm"
 			(at 141.9352 129.54 0)
 			(hide yes)
@@
 			)
 		)
-		(property "Footprint" ""
+		(property "Footprint" "Capacitor_SMD:C_0603_1608Metric"
 			(at 154.6352 129.54 0)
 			(hide yes)
@@
 			)
 		)
-		(property "Footprint" ""
+		(property "Footprint" "Resistor_SMD:R_0603_1608Metric"
 			(at 239.522 127 90)
 			(hide yes)
@@
 			)
 		)
-		(property "Footprint" ""
+		(property "Footprint" "Capacitor_THT:CP_Radial_D6.3mm_P2.50mm"
 			(at 107.6452 129.54 0)
 			(hide yes)
@@
 			)
 		)
-		(property "Footprint" ""
+		(property "Footprint" "Capacitor_SMD:C_0603_1608Metric"
 			(at 120.3452 129.54 0)
 			(hide yes)
@@
 			)
 		)
-		(property "Footprint" ""
+		(property "Footprint" "Connector_Wire:SolderWire-1sqmm_1x01_D1.4mm_OD2.7mm"
 			(at 64.77 125.73 0)
 			(hide yes)
@@
 			)
 		)
-		(property "Footprint" ""
+		(property "Footprint" "Capacitor_SMD:C_1206_3216Metric"
 			(at 237.1852 67.31 0)
 			(hide yes)
@@
 			)
 		)
-		(property "Footprint" ""
+		(property "Footprint" "Connector_Wire:SolderWire-1sqmm_1x02_P5.4mm_D1.4mm_OD2.7mm"
 			(at 124.46 20.32 0)
 			(hide yes)
@@
 			)
 		)
-		(property "Footprint" ""
+		(property "Footprint" "Connector_PinHeader_2.54mm:PinHeader_1x02_P2.54mm_Vertical"
 			(at 241.3 144.78 0)
 			(hide yes)
@@
 			)
 		)
-		(property "Footprint" ""
+		(property "Footprint" "Connector_PinHeader_2.00mm:PinHeader_1x01_P2.00mm_Vertical"
 			(at 106.68 76.2 0)
 			(hide yes)
@@
 			)
 		)
-		(property "Footprint" ""
+		(property "Footprint" "Resistor_THT:R_Axial_DIN0207_L6.3mm_D2.5mm_P10.16mm_Horizontal"
 			(at 177.8 114.808 90)
 			(hide yes)
@@
 			)
 		)
-		(property "Footprint" ""
+		(property "Footprint" "Capacitor_THT:CP_Radial_D8.0mm_P3.50mm"
 			(at 42.8752 129.54 0)
 			(hide yes)
@@
 			)
 		)
-		(property "Footprint" ""
+		(property "Footprint" "Connector_Wire:SolderWire-1sqmm_1x01_D1.4mm_OD2.7mm"
 			(at 81.28 113.03 0)
 			(hide yes)
@@
 			)
 		)
-		(property "Footprint" ""
+		(property "Footprint" "Connector_Wire:SolderWire-1sqmm_1x02_P5.4mm_D1.4mm_OD2.7mm"
 			(at 91.44 20.32 0)
 			(hide yes)
@@
 			)
 		)
-		(property "Footprint" ""
+		(property "Footprint" "Capacitor_THT:CP_Radial_D6.3mm_P2.50mm"
 			(at 249.8852 67.31 0)
 			(hide yes)
@@
 			)
 		)
-		(property "Footprint" ""
+		(property "Footprint" "Capacitor_SMD:C_0603_1608Metric"
 			(at 150.8252 67.31 0)
 			(hide yes)
@@
 			)
 		)
-		(property "Footprint" "Connector_PinHeader_2.00mm:PinHeader_1x01_P2.00mm_Vertical"
+		(property "Footprint" "Connector_Wire:SolderWire-1sqmm_1x01_D1.4mm_OD2.7mm"
 			(at 64.77 113.03 0)
 			(hide yes)
@@
 	)
 	(symbol
+		(lib_id "power:PWR_FLAG")
+		(at 95.25 171.45 180)
+		(unit 1)
+		(body_style 1)
+		(exclude_from_sim no)
+		(in_bom yes)
+		(on_board yes)
+		(in_pos_files yes)
+		(dnp no)
+		(fields_autoplaced yes)
+		(property "Reference" "#FLG07"
+			(at 95.25 173.355 0)
+			(hide yes)
+			(show_name no)
+			(do_not_autoplace no)
+			(effects
+				(font
+					(size 1.27 1.27)
+				)
+			)
+		)
+		(property "Value" "PWR_FLAG"
+			(at 95.25 176.53 0)
+			(show_name no)
+			(do_not_autoplace no)
+			(effects
+				(font
+					(size 1.27 1.27)
+				)
+			)
+		)
+		(property "Footprint" ""
+			(at 95.25 171.45 0)
+			(hide yes)
+			(show_name no)
+			(do_not_autoplace no)
+			(effects
+				(font
+					(size 1.27 1.27)
+				)
+			)
+		)
+		(property "Datasheet" ""
+			(at 95.25 171.45 0)
+			(hide yes)
+			(show_name no)
+			(do_not_autoplace no)
+			(effects
+				(font
+					(size 1.27 1.27)
+				)
+			)
+		)
+		(property "Description" "Special symbol for telling ERC where power comes from"
+			(at 95.25 171.45 0)
+			(hide yes)
+			(show_name no)
+			(do_not_autoplace no)
+			(effects
+				(font
+					(size 1.27 1.27)
+				)
+			)
+		)
+		(pin "1"
+		)
+		(instances
+			(project "PCB"
+				(path "/8904b003-95b6-476e-93a4-c0afb2c5d7e3/bd481dc0-0e8b-4283-b170-81e53db339ca"
+					(reference "#FLG07")
+					(unit 1)
+				)
+			)
+		)
+	)
+	(symbol
 		(lib_id "Connector_Generic:Conn_01x02")
 		(at 60.96 62.23 270)
@@
 			)
 		)
-		(property "Footprint" ""
+		(property "Footprint" "Capacitor_SMD:C_1206_3216Metric"
 			(at 167.3352 129.54 0)
 			(hide yes)
@@
 			)
 		)
-		(property "Footprint" ""
+		(property "Footprint" "Resistor_SMD:R_0603_1608Metric"
 			(at 87.63 168.148 90)
 			(hide yes)
@@
 			)
 		)
-		(property "Footprint" ""
+		(property "Footprint" "Connector_PinHeader_2.00mm:PinHeader_1x01_P2.00mm_Vertical"
 			(at 82.55 76.2 0)
 			(hide yes)
@@
 			)
 		)
-		(property "Footprint" ""
+		(property "Footprint" "Capacitor_SMD:C_0805_2012Metric"
 			(at 79.7052 180.34 0)
 			(hide yes)
@@
 			)
 		)
-		(property "Footprint" ""
+		(property "Footprint" "Capacitor_SMD:C_1206_3216Metric"
 			(at 162.2552 67.31 0)
 			(hide yes)
@@
 			)
 		)
-		(property "Footprint" ""
+		(property "Footprint" "Connector_PinHeader_2.00mm:PinHeader_1x01_P2.00mm_Vertical"
 			(at 81.28 50.8 0)
 			(hide yes)
@@
 			)
 		)
-		(property "Footprint" ""
+		(property "Footprint" "Connector_Wire:SolderWire-1sqmm_1x01_D1.4mm_OD2.7mm"
 			(at 81.28 125.73 0)
 			(hide yes)
@@
 			)
 		)
-		(property "Footprint" ""
+		(property "Footprint" "Connector_PinHeader_2.00mm:PinHeader_1x01_P2.00mm_Vertical"
 			(at 30.48 76.2 0)
 			(hide yes)
@@
 			)
 		)
-		(property "Footprint" ""
+		(property "Footprint" "Inductor_SMD:L_Bourns_SRR1260"
 			(at 129.54 113.03 0)
 			(hide yes)
@@
 			)
 		)
-		(property "Footprint" ""
+		(property "Footprint" "Capacitor_SMD:C_0805_2012Metric"
 			(at 39.0652 180.34 0)
 			(hide yes)
